File: PCB/PDU_v2/PDU_v2.kicad_pcb (KiCad board)
At the start: 4 copper layers, 57.6 x 60.8 mm, 58 parts, among them J1 Conn_01x02_Pin, J14 Conn_01x04_Pin, J2 Conn_01x02_Pin, J3 Conn_01x02_Pin, J4 Conn_01x02_Pin, J5 Conn_01x02_Pin, J6 Conn_01x02_Pin, J7 Conn_01x02_Pin, U1 TPS54360BQDDAQ1, U2 INA240A2D

Commit message: Started working on v2
Parts:
- removed D3: SS34, Diode_SMD:D_SMA
- added C31: 100u, Capacitor_SMD:CP_Elec_8x10, F.Cu at (178.6, 133.6)
- added C32: 100u, Capacitor_SMD:CP_Elec_8x10, F.Cu at (188.4, 133.6)
- added D4: B560C-13-F, Diode_SMD:D_SMC, F.Cu at (157.7, 46.5)
- added L1: 8.2uH, Inductor_SMD:L_Coilcraft_XAL6060-XXX, F.Cu at (156.2, 123.8)
- C1, C5: value 2.2uF -> 2u2
- C10, C11, C12, C13, C14, C15, C22, C23, C24, C25, C26, C27: footprint Capacitor_SMD:C_0805_2012Metric_Pad1.18x1.45mm_HandSolder -> Capacitor_SMD:C_1210_3225Metric_Pad1.33x2.70mm_HandSolder; moved to B.Cu
- C16, C21: value 100n -> 1u
- C18, C8: value 220u -> 470u
- C2: value 6800pF -> 6800p
- C3: value 0.1uF -> 100n
- C4, C7: value 47uF -> 47u
- C6: value 39pF -> 39p
- J1, J2, J3, J4, J5, J6, J7: value Conn_01x02_Pin -> XT60PW-M; footprint Connector_AMASS:AMASS_XT60PW-M_1x02_P7.20mm_Horizontal -> SamacSys_Parts:XT60PWM
- L2: value 8.2uH -> 8u2
- moved C26 129.8 mm to (183.4, 48.0), turned to 180 degrees
- moved C15 119.2 mm to (131.1, 44.1)
- moved C10 116.7 mm to (183.4, 51.1), turned to 180 degrees
- moved C25 112.5 mm to (131.1, 47.4)
- moved C11 104.6 mm to (183.4, 69.3), turned to 180 degrees
- moved C22 104.2 mm to (183.4, 66.1), turned to 180 degrees
- moved C24 94.8 mm to (131.2, 62.2)
- moved C12 93.2 mm to (183.4, 87.5), turned to 180 degrees
- moved C13 92.2 mm to (131.2, 65.4)
- moved C27 82.3 mm to (183.4, 84.3), turned to 180 degrees
- moved C14 77.1 mm to (131.2, 83.6)
- moved C23 73.6 mm to (131.2, 80.4)
- moved J2 72.8 mm to (178.5, 44.0), turned to -90 degrees
- moved J5 59.6 mm to (136.0, 87.5), turned to 90 degrees
- moved C20 53.6 mm to (168.7, 133.6), turned to 90 degrees
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Connections:
- C1 pad 1: VBAT -> Net-(U1-VIN)
- C10 pad 2: VBAT -> +BATT
- C11 pad 2: VBAT -> +BATT
- C12 pad 2: VBAT -> +BATT
- C13 pad 2: VBAT -> +BATT
- C14 pad 2: VBAT -> +BATT
- C15 pad 2: VBAT -> +BATT
- C16 pad 2: /SH_IN -> +BATT
- C17 pad 1: VBAT -> +BATT
- C18 pad 1: VBAT -> +BATT
- C19 pad 1: VBAT -> +BATT
- C20 pad 1: VBAT -> +BATT
- C21 pad 2: VBAT -> +BATT
- C22 pad 2: VBAT -> +BATT
- C23 pad 2: VBAT -> +BATT
- C24 pad 2: VBAT -> +BATT
- C25 pad 2: VBAT -> +BATT
- C26 pad 2: VBAT -> +BATT
- C27 pad 2: VBAT -> +BATT
- C5 pad 1: VBAT -> Net-(U1-VIN)
- C8 pad 1: VBAT -> +BATT
- C9 pad 2: VBAT -> +BATT
- J2 pad 1: VBAT -> +BATT
- J3 pad 1: VBAT -> +BATT
- J4 pad 1: VBAT -> +BATT
- J5 pad 1: VBAT -> +BATT
- J6 pad 1: VBAT -> +BATT
- J7 pad 1: VBAT -> +BATT
- R5 pad 2: VBAT -> +BATT
- R7 pad 2: VBAT -> +BATT
- R9 pad 2: VBAT -> +BATT
- U1 pad 2: VBAT -> Net-(U1-VIN)
- U2 pad 1: VBAT -> +BATT
Routing:
- net VBAT: track 10.7 -> 0.00 mm
- net +BATT: track 0.00 -> 6.06 mm
- net Net-(U1-RT/CLK): track 1.81 -> 4.76 mm
- net Net-(U1-VIN): track 0.00 -> 2.66 mm
- net (no net): track 0.00 -> 1.99 mm
- net /SW: track 1.55 -> 0.00 mm
- added copper zone on F.Cu, net Net-(U1-VIN)
- removed copper zone on F.Cu, net VBAT
Other:
- board size 57.6 x 60.8 mm -> 67.6 x 60.8 mm

Commit message: Finished layout
Parts:
- removed C3: 100n, Capacitor_SMD:C_0805_2012Metric_Pad1.18x1.45mm_HandSolder
- removed D4: B560C-13-F, Diode_SMD:D_SMC
- removed F3: Fuse, Fuse:Fuse_2920_7451Metric_Pad2.10x5.45mm_HandSolder
- removed L2: 8u2, Inductor_SMD:L_Coilcraft_XAL6060-XXX
- removed R5: 147k, Resistor_SMD:R_0603_1608Metric_Pad0.98x0.95mm_HandSolder
- removed R6: 33k, Resistor_SMD:R_0603_1608Metric_Pad0.98x0.95mm_HandSolder
- removed U1: TPS54360BQDDAQ1, Package_SO:TI_SO-PowerPAD-8_ThermalVias
- added C33: 10u, Capacitor_SMD:C_1210_3225Metric_Pad1.33x2.70mm_HandSolder, F.Cu at (172.9, 39.8)
- added C34: 10u, Capacitor_SMD:C_1210_3225Metric_Pad1.33x2.70mm_HandSolder, F.Cu at (172.9, 70.1)
- added C35: 10u, Capacitor_SMD:C_1210_3225Metric_Pad1.33x2.70mm_HandSolder, F.Cu at (172.9, 91.7)
- added C36: 10u, Capacitor_SMD:C_1210_3225Metric_Pad1.33x2.70mm_HandSolder, F.Cu at (172.9, 65.8)
- added C37: 10u, Capacitor_SMD:C_1210_3225Metric_Pad1.33x2.70mm_HandSolder, F.Cu at (172.9, 61.4)
- added C38: 10u, Capacitor_SMD:C_1210_3225Metric_Pad1.33x2.70mm_HandSolder, F.Cu at (172.9, 44.2)
- added C39: 10u, Capacitor_SMD:C_1210_3225Metric_Pad1.33x2.70mm_HandSolder, F.Cu at (172.9, 74.5)
- added C40: 10u, Capacitor_SMD:C_1210_3225Metric_Pad1.33x2.70mm_HandSolder, F.Cu at (172.9, 87.3)
- added C41: 10u, Capacitor_SMD:C_1210_3225Metric_Pad1.33x2.70mm_HandSolder, F.Cu at (172.9, 57.0)
- added C42: 10u, Capacitor_SMD:C_1210_3225Metric_Pad1.33x2.70mm_HandSolder, F.Cu at (141.6, 87.3)
- added C43: 10u, Capacitor_SMD:C_1210_3225Metric_Pad1.33x2.70mm_HandSolder, F.Cu at (141.6, 61.4)
- added F1: SF-2923HC30C-2, SamacSys_Parts:SF2923HC30C2, F.Cu at (149.6, 76.3)
- added IC1: LMR51635YFDDCR, SamacSys_Parts:SOT95P280X110-6N, F.Cu at (152.7, 44.9)
- added L3: 18u, Inductor_SMD:L_Coilcraft_XAL6060-XXX, F.Cu at (159.0, 46.7)
- C16, C21: value 1u -> 10u; footprint Capacitor_SMD:C_0805_2012Metric_Pad1.18x1.45mm_HandSolder -> Capacitor_SMD:C_1210_3225Metric_Pad1.33x2.70mm_HandSolder
- C19, C20, C31, C32: value 100u -> 10u; footprint Capacitor_SMD:CP_Elec_8x10 -> Capacitor_SMD:C_1210_3225Metric_Pad1.33x2.70mm_HandSolder
- C2: value 6800p -> 100n
- C28: value 0.1uF -> 100n; footprint Capacitor_SMD:C_0805_2012Metric_Pad1.18x1.45mm_HandSolder -> Capacitor_SMD:C_0603_1608Metric_Pad1.08x0.95mm_HandSolder; moved to B.Cu
- C29: value 1uF -> 1u; moved to B.Cu
- C4: value 47u -> 33u; footprint Capacitor_SMD:C_0805_2012Metric_Pad1.18x1.45mm_HandSolder -> Capacitor_SMD:C_1210_3225Metric_Pad1.33x2.70mm_HandSolder
- C6: value 39p -> 33u; footprint Capacitor_SMD:C_0805_2012Metric_Pad1.18x1.45mm_HandSolder -> Capacitor_SMD:C_1210_3225Metric_Pad1.33x2.70mm_HandSolder
- C7: value 47u -> 100n
- C9: value 100n -> 10u; footprint Capacitor_SMD:C_0805_2012Metric_Pad1.18x1.45mm_HandSolder -> Capacitor_SMD:C_1210_3225Metric_Pad1.33x2.70mm_HandSolder
- L1: value 8.2uH -> 2u2; footprint Inductor_SMD:L_Coilcraft_XAL6060-XXX -> SamacSys_Parts:WE-MAPI_4020
- R1: value 162k -> 68k
- R3: value 68k -> 0R
- R4: value 13k -> DNP
- R7: value R -> 0m5; footprint Resistor_SMD:R_Shunt_Vishay_WSR2_WSR3 -> Resistor_SMD:R_2512_6332Metric_Pad1.40x3.35mm_HandSolder
- R8, U2: moved to B.Cu
- moved C32 101.0 mm to (141.6, 44.2), turned to 180 degrees
- moved C20 97.7 mm to (141.6, 39.8), turned to 180 degrees
- moved C31 85.1 mm to (141.6, 57.0), turned to 180 degrees
- moved R10 80.0 mm to (147.3, 38.4)
- moved R9 79.8 mm to (145.8, 38.4), turned to -90 degrees
- moved C30 78.6 mm to (149.0, 38.5)
- moved C8 76.4 mm to (157.3, 62.5)
- moved C18 73.2 mm to (166.1, 62.5)
- moved C17 71.7 mm to (148.5, 62.5)
- moved L1 71.3 mm to (148.0, 53.0), turned to 0 degrees
- moved C19 61.6 mm to (141.6, 74.5), turned to 180 degrees
- moved U2 58.7 mm to (159.0, 65.9), turned to 180 degrees
- moved C9 57.5 mm to (141.6, 70.1), turned to 180 degrees
- moved C28 56.4 mm to (154.6, 65.7), turned to -90 degrees
- moved C21 56.4 mm to (141.6, 65.8), turned to 180 degrees
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Connections:
- net /BAT_IN renamed +VBATT_IN
- net Net-(U1-FB) renamed /EN_BK
- C1 pad 1: Net-(U1-VIN) -> /VIN_BK
- C19 pad 1: +BATT -> GND
- C19 pad 2: GND -> +BATT
- C2 pad 1: Net-(C2-Pad1) -> /CB_BK
- C2 pad 2: GND -> /SW_BK
- C20 pad 1: +BATT -> GND
- C20 pad 2: GND -> +BATT
- C31 pad 1: Net-(U1-VIN) -> GND
- C31 pad 2: GND -> +BATT
- C32 pad 1: +BATT -> GND
- C32 pad 2: GND -> +BATT
- C5 pad 1: Net-(U1-VIN) -> /VIN_BK
- C6 pad 1: Net-(U1-COMP) -> 5V
- C7 pad 1: 5V -> /VIN_BK
- J14 pad 2: BAT_VOL -> BAT_CURR
- J14 pad 4: BAT_CURR -> BAT_VOL
- L1 pad 2: Net-(U1-VIN) -> /VIN_BK
- R1 pad 1: GND -> 5V
- R1 pad 2: Net-(U1-RT/CLK) -> /FB_BK
- R2 pad 1: Net-(U1-COMP) -> /FB_BK
- R2 pad 2: Net-(C2-Pad1) -> GND
- R3 pad 1: 5V -> /VIN_BK
Routing:
- net BAT_CURR: track 0.00 -> 29.4 mm
- net 5V: track 13.4 -> 28.4 mm, vias 0 -> 1
- net BAT_VOL: track 0.00 -> 7.93 mm
- net Net-(R8-Pad2): track 0.00 -> 7.52 mm
- net +BATT: track 6.06 -> 12.2 mm, vias 0 -> 1
- net /SH_IN: track 6.14 -> 12.0 mm, vias 0 -> 1
- net GND: track 15.5 -> 10.1 mm, vias 0 -> 3
- net TPS_EN: track 4.95 -> 0.00 mm
- net Net-(U1-RT/CLK): track 4.76 -> 0.00 mm
- net Net-(U1-COMP): track 4.30 -> 0.00 mm
- net /EN_BK: track 3.26 -> 0.00 mm
- net Net-(U1-VIN): track 2.66 -> 0.00 mm
- net (no net): track 1.99 -> 0.00 mm
- net Net-(U1-BOOT): track 1.91 -> 0.00 mm
- net Net-(C2-Pad1): track 1.71 -> 0.00 mm
- added copper zone on F.Cu, net +BATT
- added copper zone on In2.Cu, net +BATT
- added copper zone on F.Cu, net /SW_BK
- added copper zone on F.Cu, net /VIN_BK
- added copper zone on F.Cu, net GND
- removed copper zone on F.Cu, net /SW
- removed copper zone on F.Cu, net Net-(U1-VIN)

Commit message: Repaired library
Parts:
- removed J2, J3, J4, J5, J6, J7: XT60PW-M, SamacSys_Parts:XT60PWM
- added D3: LED_P1, LED_SMD:LED_0805_2012Metric_Pad1.15x1.40mm_HandSolder, F.Cu at (167.7, 38.9)
- added PS1: XT60PW-M, SamacSys_Parts:XT60PWM, F.Cu at (153.6, 86.1)
- added PS2: XT60PW-M, SamacSys_Parts:XT60PWM, F.Cu at (178.7, 87.8)
- added PS3: XT60PW-M, SamacSys_Parts:XT60PWM, F.Cu at (178.7, 69.3)
- added PS4: XT60PW-M, SamacSys_Parts:XT60PWM, F.Cu at (178.7, 50.8)
- added PS5: XT60PW-M, SamacSys_Parts:XT60PWM, F.Cu at (135.8, 43.6)
- added PS6: XT60PW-M, SamacSys_Parts:XT60PWM, F.Cu at (135.8, 62.1)
- added PS7: XT60PW-M, SamacSys_Parts:XT60PWM, F.Cu at (135.8, 80.7)
- added R5: 2k, Resistor_SMD:R_0603_1608Metric_Pad0.98x0.95mm_HandSolder, F.Cu at (167.7, 40.8)
- moved F1 0.52 mm to (150.1, 76.1)
Connections:
- net +BATT renamed SH_OUT
- net /SH_IN renamed SH_IN
- net 5V renamed +5V
Routing:
- net unconnected-(J1-MH1-Pad3): vias 0 -> 1

Commit message: layout update
Routing:
- net GND: track 10.1 -> 40.0 mm, vias 3 -> 49
- net /FB_BK: track 0.00 -> 3.70 mm
- net /EN_BK: track 0.00 -> 3.70 mm
- net +5V: track 28.4 -> 31.8 mm
- net Net-(D3-A): track 0.00 -> 1.91 mm
- added copper zone on B.Cu, net SH_OUT
